Commit message: added fake bridge and remove debug visual

File: xela_models/urdf/xela.xacro (robot description, xacro)
@@ -43,5 +43,5 @@
     </link>
     <link name="${sequence}_base2x">
-      <visual>
+      <!-- <visual>
         <geometry>
           <sphere radius="0.0001"/>
@@ -49,5 +49,5 @@
         <origin xyz="${x} ${y} ${z}" rpy="0 0 0"/>
         <material name="${col}"/>
-      </visual>
+      </visual>  -->
       <collision>
         <geometry>
@@ -57,5 +57,5 @@
     </link>
     <link name="${sequence}_x2y">
-      <visual>
+      <!-- <visual>
         <geometry>
           <sphere radius="0.0001"/>
@@ -63,5 +63,5 @@
         <origin xyz="0.0 0.0 0.0" rpy="0 0 0"/>
         <material name="${col}"/>
-      </visual>
+      </visual>  -->
       <collision>
         <geometry>
